Commit message: Add mapping launch package

File: src/grobot_description/urdf/grobot.urdf.xacro (robot description, xacro)
@@ -30,10 +30,4 @@
     <color rgba="0.05 0.25 0.75 1.0"/>
   </material>
-  <link name="base_footprint"/>
-  <joint name="base_footprint_joint" type="fixed">
-    <parent link="base_footprint"/>
-    <child link="base_link"/>
-    <origin xyz="0 0 ${wheel_radius}" rpy="0 0 0"/>
-  </joint>
   <link name="base_link">
     <visual>

Commit message: Fix Nav2 bringup launch

File: src/grobot_description/urdf/grobot.urdf.xacro (robot description, xacro)
@@ -45,4 +45,10 @@
     </collision>
   </link>
+  <link name="base_footprint"/>
+  <joint name="base_footprint_joint" type="fixed">
+    <parent link="base_link"/>
+    <child link="base_footprint"/>
+    <origin xyz="0 0 0" rpy="0 0 0"/>
+  </joint>
   <link name="left_wheel_link">
     <visual>

Commit message: Update robot geometry parameters

File: src/grobot_description/urdf/grobot.urdf.xacro (robot description, xacro)
@@ -1,16 +1,15 @@
 <?xml version="1.0"?>
 <robot xmlns:xacro="http://www.ros.org/wiki/xacro" name="grobot">
-  <xacro:arg name="base_length" default="0.60"/>
-  <xacro:arg name="base_width" default="0.45"/>
+  <xacro:arg name="base_diameter" default="0.505"/>
   <xacro:arg name="base_height" default="0.18"/>
   <xacro:arg name="wheel_radius" default="0.085"/>
   <xacro:arg name="wheel_width" default="0.045"/>
   <xacro:arg name="track_width" default="0.375"/>
-  <xacro:arg name="lidar_x" default="0.0"/>
+  <xacro:arg name="lidar_x" default="0.18"/>
   <xacro:arg name="lidar_y" default="0.0"/>
-  <xacro:arg name="lidar_z" default="0.20"/>
+  <xacro:arg name="lidar_z" default="0.05"/>
   <xacro:arg name="lidar_yaw" default="0.0"/>
-  <xacro:property name="base_length" value="${float('$(arg base_length)')}"/>
-  <xacro:property name="base_width" value="${float('$(arg base_width)')}"/>
+  <xacro:property name="base_diameter" value="${float('$(arg base_diameter)')}"/>
+  <xacro:property name="base_radius" value="${base_diameter / 2.0}"/>
   <xacro:property name="base_height" value="${float('$(arg base_height)')}"/>
   <xacro:property name="wheel_radius" value="${float('$(arg wheel_radius)')}"/>
@@ -34,5 +33,5 @@
       <origin xyz="0 0 0" rpy="0 0 0"/>
       <geometry>
-        <box size="${base_length} ${base_width} ${base_height}"/>
+        <cylinder radius="${base_radius}" length="${base_height}"/>
       </geometry>
       <material name="body_gray"/>
@@ -41,5 +40,5 @@
       <origin xyz="0 0 0" rpy="0 0 0"/>
       <geometry>
-        <box size="${base_length} ${base_width} ${base_height}"/>
+        <cylinder radius="${base_radius}" length="${base_height}"/>
       </geometry>
     </collision>

Commit message: 集成 IMU 驱动，slam_toolbox 启用 IMU 融合
- 迁移 wit_ros2_imu 和 imu_msg 包到项目中
- 修复 wit_ros2_imu 的 package.xml 依赖声明
- 新增 grobot_bringup/config/imu_params.yaml 参数配置
- 新增 grobot_bringup/launch/imu.launch.py 启动文件
- robot.launch.py 集成 IMU 启动（ros2 launch grobot_bringup robot.launch.py 自动启动 IMU）
- robot_description 添加 imu_link 及安装位姿参数
- slam_toolbox.yaml 启用 use_imu_data + imu_topic

File: src/grobot_description/urdf/grobot.urdf.xacro (robot description, xacro)
@@ -10,4 +10,10 @@
   <xacro:arg name="lidar_z" default="0.05"/>
   <xacro:arg name="lidar_yaw" default="0.0"/>
+  <xacro:arg name="imu_x" default="0.0"/>
+  <xacro:arg name="imu_y" default="0.0"/>
+  <xacro:arg name="imu_z" default="0.10"/>
+  <xacro:arg name="imu_roll" default="0.0"/>
+  <xacro:arg name="imu_pitch" default="0.0"/>
+  <xacro:arg name="imu_yaw" default="0.0"/>
   <xacro:property name="base_diameter" value="${float('$(arg base_diameter)')}"/>
   <xacro:property name="base_radius" value="${base_diameter / 2.0}"/>
@@ -20,4 +26,10 @@
   <xacro:property name="lidar_z" value="${float('$(arg lidar_z)')}"/>
   <xacro:property name="lidar_yaw" value="${float('$(arg lidar_yaw)')}"/>
+  <xacro:property name="imu_x" value="${float('$(arg imu_x)')}"/>
+  <xacro:property name="imu_y" value="${float('$(arg imu_y)')}"/>
+  <xacro:property name="imu_z" value="${float('$(arg imu_z)')}"/>
+  <xacro:property name="imu_roll" value="${float('$(arg imu_roll)')}"/>
+  <xacro:property name="imu_pitch" value="${float('$(arg imu_pitch)')}"/>
+  <xacro:property name="imu_yaw" value="${float('$(arg imu_yaw)')}"/>
   <material name="body_gray">
     <color rgba="0.35 0.38 0.42 1.0"/>
@@ -92,3 +104,17 @@
     <origin xyz="${lidar_x} ${lidar_y} ${lidar_z}" rpy="0 0 ${lidar_yaw}"/>
   </joint>
+  <link name="imu_link">
+    <visual>
+      <origin xyz="0 0 0" rpy="0 0 0"/>
+      <geometry>
+        <box size="0.03 0.03 0.02"/>
+      </geometry>
+      <material name="lidar_blue"/>
+    </visual>
+  </link>
+  <joint name="imu_joint" type="fixed">
+    <parent link="base_link"/>
+    <child link="imu_link"/>
+    <origin xyz="${imu_x} ${imu_y} ${imu_z}" rpy="${imu_roll} ${imu_pitch} ${imu_yaw}"/>
+  </joint>
 </robot>
